File: HW/OCTO_CONTROLER_V1.1.sch (EAGLE design)
At the start: 44 parts, among them IC1 N-DUAL-FET, IC2 N-DUAL-FET, IC3 CXDM4060P, IC4 AOZ1284PI, J1 DC_POWER, Q1 DTC114EUA, Q2 CXDM4060P, Q3 DTC114EUA, X1 RASPI_BOARD_B+#_F

Commit message: v1.1 pcb gerber
Parts:
- JP1: value STRIP LED -> ECH350R
- JP2: value DC-IN -> ECH350R
- JP3, JP4: value MA02ECH350R -> ECH350R
Other:
- note added: "(DC12V or DC24V ADAPTER USED)"
- note added: "(DC12V or DC24V LED STRIP)"
- note added: "(DC12V or DC24V RELAY USED)"
- note added: "CONNECTOR->RELAY -> PSU CONTROL"
- note added: "DC 5V OUT"
- note added: "DC POWER INPUT"
- note added: "DC7~35V Input range(DC 12V or DC24V)"
- note added: "LED POWER"
- note added: "LED STRIP"
- note added: "MAXIMUM 5V 4A OUT"
- note added: "OCTO PRINTER CONTROLER V1.1"
- note added: "PSU CONTROL"
- note removed: "(12V OR 24V)"
- note removed: "3D PRINTER EXTERNAL POWER RELAY"
- note removed: "DC7~35V Input"
- note removed: "Max 4A"
- note removed: "OCTO PRINTER CONTROLER V1.0"
- note removed: "REGULATOR"
Changed lines of the file:
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@@
 <part name="R8" library="cona_lib" deviceset="R_" device="0603" value="11k"/>
 <part name="C1" library="cona_lib" deviceset="C_" device="3225" value="10uF/35V"/>
-<part name="JP2" library="cona_lib" deviceset="MA02" device="ECH350R" value="DC-IN"/>
+<part name="JP2" library="cona_lib" deviceset="MA02" device="ECH350R" value="ECH350R"/>
 <part name="SUPPLY6" library="supply2" deviceset="VEE" device=""/>
 <part name="IC3" library="cona_lib" deviceset="CXDM4060P" device="CXDM4060P" value="CXDM4060P"/>
 <part name="R5" library="cona_lib" deviceset="R_" device="0603" value="100kF"/>
 <part name="ZD3" library="GRU-EURO6" deviceset="ZENER_DIODE" device="RD47S" value="RD10S"/>
-<part name="JP3" library="cona_lib" deviceset="MA02" device="ECH350R"/>
+<part name="JP3" library="cona_lib" deviceset="MA02" device="ECH350R" value="ECH350R"/>
 <part name="PE5" library="cona_lib" deviceset="GND" device=""/>
 <part name="R6" library="cona_lib" deviceset="R_" device="0603" value="200"/>
@@
 <part name="SUPPLY1" library="supply2" deviceset="VEE" device=""/>
 <part name="LED2" library="cona_lib" deviceset="LED" device="3FG2HD-T1" value="STATUS"/>
-<part name="JP1" library="cona_lib" deviceset="MA04-1" device="ECHR350R" value="STRIP LED"/>
+<part name="JP1" library="cona_lib" deviceset="MA04-1" device="ECHR350R" value="ECH350R"/>
 <part name="IC1" library="cona_lib" deviceset="N-DUAL-FET" device=""/>
 <part name="PE1" library="cona_lib" deviceset="GND" device=""/>
@@
 <part name="JP5" library="cona_lib" deviceset="SERVO-3CH" device=""/>
 <part name="+3V3" library="cona_lib" deviceset="+3V3" device=""/>
-<part name="JP4" library="cona_lib" deviceset="MA02" device="ECH350R"/>
+<part name="JP4" library="cona_lib" deviceset="MA02" device="ECH350R" value="ECH350R"/>
 <part name="P+1" library="cona_lib" deviceset="+5V" device=""/>
 <part name="PE11" library="cona_lib" deviceset="GND" device=""/>
@@
 <sheet>
 <plain>
-<text x="-208.28" y="53.34" size="10.16" layer="97">OCTO PRINTER  CONTROLER V1.0</text>
+<text x="-208.28" y="45.72" size="10.16" layer="97">OCTO PRINTER  CONTROLER V1.1</text>
 <wire x1="-208.28" y1="-53.34" x2="-119.38" y2="-53.34" width="0.1524" layer="97"/>
 <wire x1="-208.28" y1="-144.78" x2="-119.38" y2="-144.78" width="0.1524" layer="97"/>
@@
 <wire x1="58.42" y1="-144.78" x2="58.42" y2="-53.34" width="0.1524" layer="97"/>
 <wire x1="58.42" y1="-53.34" x2="-114.3" y2="-53.34" width="0.1524" layer="97"/>
-<text x="-58.42" y="-88.9" size="3.81" layer="97">+5 Voltage Step Down Regulator</text>
-<text x="-99.06" y="-60.96" size="1.778" layer="98" rot="MR180">DC7~35V Input</text>
-<text x="40.64" y="-99.06" size="1.778" layer="98" rot="MR180">Max 4A</text>
-<text x="-109.22" y="-58.42" size="3.81" layer="97">REGULATOR</text>
+<text x="-60.96" y="-81.28" size="3.81" layer="97">+5 Voltage Step Down Regulator</text>
+<text x="-99.06" y="-60.96" size="1.778" layer="98" rot="MR180">DC7~35V Input range(DC 12V or DC24V)</text>
+<text x="-109.22" y="-58.42" size="3.81" layer="97">DC POWER INPUT</text>
 <text x="15.24" y="-106.68" size="1.778" layer="98" rot="MR180">Vo = 0.8*(1+R37/R38)</text>
 <text x="2.54" y="-91.44" size="1.778" layer="98" rot="MR180">FSW R : 100K = 500kHz</text>
 <text x="2.54" y="-93.98" size="1.778" layer="98" rot="MR180">FSW R : 270K = 200kHz</text>
 <text x="2.54" y="-96.52" size="1.778" layer="98" rot="MR180">FSW R : 46.6k = 1MHz</text>
-<text x="-45.72" y="7.62" size="3.81" layer="97" rot="MR180">3D PRINTER EXTERNAL POWER RELAY</text>
+<text x="-45.72" y="7.62" size="3.81" layer="97" rot="MR180">PSU CONTROL</text>
 <text x="-111.76" y="33.02" size="3.81" layer="97">STATUS LED</text>
 <wire x1="-114.3" y1="38.1" x2="-114.3" y2="-50.8" width="0.1524" layer="97"/>
@@
 <wire x1="58.42" y1="-50.8" x2="58.42" y2="10.16" width="0.1524" layer="97"/>
 <text x="-109.22" y="-12.7" size="3.81" layer="97">OPTION I/O</text>
-<text x="-45.72" y="2.54" size="3.81" layer="97" rot="MR180">(12V OR 24V)</text>
+<text x="-205.74" y="-58.42" size="3.81" layer="97">LED STRIP</text>
+<text x="27.94" y="-71.12" size="3.81" layer="97">DC 5V OUT</text>
+<text x="-43.18" y="-45.72" size="1.778" layer="98" rot="MR90">CONNECTOR-&gt;RELAY -&gt; PSU CONTROL</text>
+<text x="-175.26" y="-55.88" size="1.778" layer="98" rot="MR180">(DC12V or DC24V LED STRIP)</text>
+<text x="-58.42" y="-55.88" size="1.778" layer="98" rot="MR180">(DC12V or DC24V  ADAPTER USED)</text>
+<text x="-2.54" y="5.08" size="1.778" layer="98" rot="MR180">(DC12V or DC24V RELAY USED)</text>
+<text x="-111.76" y="-91.44" size="1.778" layer="98" rot="MR180">LED POWER</text>
+<text x="-43.18" y="-83.82" size="2.54" layer="98" rot="MR180">MAXIMUM 5V 4A OUT</text>
 </plain>
 <instances>

Commit message: 거버업로드
Parts:
- removed D3: MBRS540T3, diode:DIODE-SMC
- added D1: 1N4148WS, cona_lib:B5189WN
- D2: value 1N4148WS -> MBRS540T3; device cona_lib:B5189WN -> diode:DIODE-SMC
- JP3: value ECH350R -> SERVO-3CH; device cona_lib:MA02ECH350R -> cona_lib:SERVO-3CH
- JP5: value SERVO-3CH -> ECH350R; device cona_lib:SERVO-3CH -> cona_lib:MA02ECH350R
Connections:
- net +5V: now also JP5.1; no longer JP4.1
- net 3V3: now also JP3.GND; no longer JP5.GND
- net GND: now also D1.A, JP3.+5V, JP5.2; no longer D3.A, JP3.2, JP5.+5V
- net IO1: now also JP3.1; no longer JP5.1
- net IO2: now also JP3.2; no longer JP5.2
- net IO3: now also JP3.3; no longer JP5.3
- net N$15: now also D1.C, JP4.1; no longer D2.C, JP3.1
- net N$27: now also D2.C; no longer D3.C
Other:
- moved on the sheet: D2, JP4
Changed lines of the file:
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@@
 <part name="R11" library="cona_lib" deviceset="R_" device="0603" value="47k"/>
 <part name="C3" library="cona_lib" deviceset="C_" device="0603" value="0.1uF/50V"/>
-<part name="D3" library="diode" deviceset="DIODE-" device="SMC" value="MBRS540T3"/>
+<part name="D2" library="diode" deviceset="DIODE-" device="SMC" value="MBRS540T3"/>
 <part name="R7" library="cona_lib" deviceset="R_" device="0603" value="47k"/>
 <part name="C7" library="cona_lib" deviceset="C_" device="0603" value="0.1uF"/>
@@
 <part name="R5" library="cona_lib" deviceset="R_" device="0603" value="100kF"/>
 <part name="ZD3" library="GRU-EURO6" deviceset="ZENER_DIODE" device="RD47S" value="RD10S"/>
-<part name="JP3" library="cona_lib" deviceset="MA02" device="ECH350R" value="ECH350R"/>
+<part name="JP4" library="cona_lib" deviceset="MA02" device="ECH350R" value="ECH350R"/>
 <part name="PE5" library="cona_lib" deviceset="GND" device=""/>
 <part name="R6" library="cona_lib" deviceset="R_" device="0603" value="200"/>
@@
 <part name="PE8" library="cona_lib" deviceset="GND" device=""/>
 <part name="PE9" library="cona_lib" deviceset="GND" device=""/>
-<part name="D2" library="cona_lib" deviceset="B5189W" device="N" value="1N4148WS"/>
+<part name="D1" library="cona_lib" deviceset="B5189W" device="N" value="1N4148WS"/>
 <part name="RN1" library="cona_lib" deviceset="4R-N" device="" value="47"/>
 <part name="LED1" library="cona_lib" deviceset="LED" device="SMD-1608" value="NC"/>
@@
 <part name="+3V1" library="cona_lib" deviceset="+3V3" device=""/>
 <part name="+3V2" library="cona_lib" deviceset="+3V3" device=""/>
-<part name="JP5" library="cona_lib" deviceset="SERVO-3CH" device=""/>
+<part name="JP3" library="cona_lib" deviceset="SERVO-3CH" device=""/>
 <part name="+3V3" library="cona_lib" deviceset="+3V3" device=""/>
-<part name="JP4" library="cona_lib" deviceset="MA02" device="ECH350R" value="ECH350R"/>
+<part name="JP5" library="cona_lib" deviceset="MA02" device="ECH350R" value="ECH350R"/>
 <part name="P+1" library="cona_lib" deviceset="+5V" device=""/>
 <part name="PE11" library="cona_lib" deviceset="GND" device=""/>
@@
 <instance part="R11" gate="G$1" x="-7.62" y="-101.6"/>
 <instance part="C3" gate="G$1" x="-43.18" y="-124.46" rot="R90"/>
-<instance part="D3" gate="G$1" x="7.62" y="-121.92" smashed="yes" rot="R90">
+<instance part="D2" gate="G$1" x="7.62" y="-121.92" smashed="yes" rot="R90">
 <attribute name="NAME" x="4.5974" y="-124.46" size="1.778" layer="95" rot="R90"/>
 <attribute name="VALUE" x="12.4714" y="-132.08" size="1.778" layer="96" rot="R90"/>
@@
 <instance part="R5" gate="G$1" x="-78.74" y="-111.76" rot="MR270"/>
 <instance part="ZD3" gate="G$1" x="-68.58" y="-101.6" rot="R90"/>
-<instance part="JP3" gate="G$1" x="-35.56" y="-30.48" rot="MR180"/>
+<instance part="JP4" gate="G$1" x="-35.56" y="-30.48" rot="MR180"/>
 <instance part="PE5" gate="M" x="-27.94" y="-40.64" rot="MR0"/>
 <instance part="R6" gate="G$1" x="-66.04" y="10.16" smashed="yes" rot="MR270">
@@
 <instance part="PE8" gate="M" x="-137.16" y="-129.54" rot="MR0"/>
 <instance part="PE9" gate="M" x="-129.54" y="-129.54" rot="MR0"/>
-<instance part="D2" gate="G$1" x="-17.78" y="-38.1" smashed="yes" rot="MR90">
+<instance part="D1" gate="G$1" x="-17.78" y="-38.1" smashed="yes" rot="MR90">
 <attribute name="NAME" x="-14.7574" y="-38.1" size="1.778" layer="95" rot="MR90"/>
 <attribute name="VALUE" x="-21.1074" y="-39.37" size="1.778" layer="96" rot="MR90"/>
@@
 <instance part="+3V1" gate="G$1" x="-147.32" y="25.4"/>
 <instance part="+3V2" gate="G$1" x="-99.06" y="-15.24"/>
-<instance part="JP5" gate="G$1" x="-93.98" y="-30.48" rot="R270"/>
+<instance part="JP3" gate="G$1" x="-93.98" y="-30.48" rot="R270"/>
 <instance part="+3V3" gate="G$1" x="-66.04" y="33.02"/>
-<instance part="JP4" gate="G$1" x="50.8" y="-88.9" rot="R180"/>
+<instance part="JP5" gate="G$1" x="50.8" y="-88.9" rot="R180"/>
 <instance part="P+1" gate="1" x="40.64" y="-73.66"/>
 <instance part="PE11" gate="M" x="40.64" y="-93.98" rot="MR0"/>
@@
 </segment>
 <segment>
-<pinref part="JP3" gate="G$1" pin="2"/>
+<pinref part="JP4" gate="G$1" pin="2"/>
 <wire x1="-30.48" y1="-30.48" x2="-27.94" y2="-30.48" width="0.1524" layer="91"/>
 <pinref part="PE5" gate="M" pin="GND"/>
@@
 </segment>
 <segment>
-<pinref part="D3" gate="G$1" pin="A"/>
+<pinref part="D2" gate="G$1" pin="A"/>
 <wire x1="7.62" y1="-127" x2="7.62" y2="-124.46" width="0.1524" layer="91"/>
 <pinref part="PE19" gate="M" pin="GND"/>
@@
 <segment>
 <pinref part="PE3" gate="M" pin="GND"/>
-<pinref part="D2" gate="G$1" pin="A"/>
+<pinref part="D1" gate="G$1" pin="A"/>
 </segment>
 <segment>
@@
 <wire x1="-86.36" y1="-15.24" x2="-86.36" y2="-17.78" width="0.1524" layer="91"/>
 <pinref part="PE10" gate="M" pin="GND"/>
-<pinref part="JP5" gate="G$1" pin="+5V"/>
-</segment>
-<segment>
-<pinref part="JP4" gate="G$1" pin="2"/>
+<pinref part="JP3" gate="G$1" pin="+5V"/>
+</segment>
+<segment>
+<pinref part="JP5" gate="G$1" pin="2"/>
 <wire x1="45.72" y1="-88.9" x2="40.64" y2="-88.9" width="0.1524" layer="91"/>
 <pinref part="PE11" gate="M" pin="GND"/>
@@
 <wire x1="-83.82" y1="-30.48" x2="-73.66" y2="-30.48" width="0.1524" layer="91"/>
 <label x="-81.28" y="-30.48" size="1.778" layer="95"/>
-<pinref part="JP5" gate="G$1" pin="2"/>
+<pinref part="JP3" gate="G$1" pin="2"/>
 </segment>
 <segment>
@@
 </segment>
 <segment>
-<pinref part="JP4" gate="G$1" pin="1"/>
+<pinref part="JP5" gate="G$1" pin="1"/>
 <pinref part="P+1" gate="1" pin="+5V"/>
 <wire x1="45.72" y1="-86.36" x2="40.64" y2="-86.36" width="0.1524" layer="91"/>
@@
 <pinref part="L1" gate="G$1" pin="2"/>
 <junction x="7.62" y="-111.76"/>
-<pinref part="D3" gate="G$1" pin="C"/>
+<pinref part="D2" gate="G$1" pin="C"/>
 <wire x1="7.62" y1="-111.76" x2="7.62" y2="-116.84" width="0.1524" layer="91"/>
 <pinref part="IC4" gate="G$1" pin="LX"/>
@@
 <segment>
 <pinref part="Q2" gate="G$1" pin="D"/>
-<pinref part="JP3" gate="G$1" pin="1"/>
+<pinref part="JP4" gate="G$1" pin="1"/>
 <wire x1="-30.48" y1="-27.94" x2="-17.78" y2="-27.94" width="0.1524" layer="91"/>
 <junction x="-17.78" y="-27.94"/>
 <wire x1="-17.78" y1="-27.94" x2="-17.78" y2="-33.02" width="0.1524" layer="91"/>
-<pinref part="D2" gate="G$1" pin="C"/>
+<pinref part="D1" gate="G$1" pin="C"/>
 </segment>
 </net>
@@
 <wire x1="-83.82" y1="-27.94" x2="-73.66" y2="-27.94" width="0.1524" layer="91"/>
 <label x="-81.28" y="-27.94" size="1.778" layer="95"/>
-<pinref part="JP5" gate="G$1" pin="1"/>
+<pinref part="JP3" gate="G$1" pin="1"/>
 </segment>
 <segment>
@@
 <pinref part="+3V2" gate="G$1" pin="3V3"/>
 <wire x1="-99.06" y1="-17.78" x2="-99.06" y2="-20.32" width="0.1524" layer="91"/>
-<pinref part="JP5" gate="G$1" pin="GND"/>
+<pinref part="JP3" gate="G$1" pin="GND"/>
 </segment>
 <segment>
@@
 <wire x1="-83.82" y1="-33.02" x2="-73.66" y2="-33.02" width="0.1524" layer="91"/>
 <label x="-81.28" y="-33.02" size="1.778" layer="95"/>
-<pinref part="JP5" gate="G$1" pin="3"/>
-</segment>
-</net>
+<pinref part="JP3" gate="G$1" pin="3"/>
+</segment>
+</net>
