File: HW/OCTO_CONTROLER_V1.2.brd (EAGLE design)
At the start: 65 x 56 mm, 44 parts, among them IC1 NTMD5838NL, IC2 NTMD5838NL, IC3 CXDM4060P, IC4 AOZ1284PI, J1 DC_POWER, Q1 DTC114EUA, Q2 CXDM4060P, Q3 DTC114EUA, X1 RASPI_BOARD_B+#_F

Commit message: BOM & V1.2 PCB UPDATE
Parts:
- added R14: 10kF, cona_lib:R0603
- added ZD4, ZD5: RD36S, GRU-EURO6:DSMM
- added ZD6: RD16S, GRU-EURO6:DSMM
- R10: value 4.7k -> 47k
- R11: value 47k -> 2k
- R12: value 52.3kF -> 2.2k
- R13: value 10kF -> 52.3kF
- R9: value 10kF -> 10k
- ZD1: value SM6T39CAY -> SM6T33CAY
- moved R12 39.6 mm to (-27.1, 3.15), turned to 270 degrees
- moved R11 28.4 mm to (-28.8, 3.15), turned to 270 degrees
- moved R10 28.3 mm to (-11.4, 25.6), turned to 90 degrees
- moved R13 3.05 mm to (-2.45, 34.1)
- moved Q3 1.50 mm to (-24.9, 3.08)
Connections:
- new net N$1: Q2.3, R11.1, R12.2, ZD6.A
- new net N$3: ZD4.A, ZD5.A
- net +5V: now also R13.2; no longer R12.2
- net GND: now also R10.2, R14.1; no longer R11.2, R13.1
- net N$12: now also R13.1, R14.2; no longer R12.1, R13.2
- net N$15: now also ZD5.C
- net N$28: now also R10.1; no longer R11.1
- net N$32: now also R12.1; no longer Q2.3, R10.1
- net VEE: now also R11.2, ZD4.C, ZD6.C; no longer R10.2
Routing:
- net VEE: track 44.6 -> 54.2 mm, vias 2 -> 4
- net N$1: track 0.00 -> 6.50 mm
- net N$15: track 13.9 -> 18.0 mm
- net N$32: track 4.18 -> 2.23 mm
- net N$3: track 0.00 -> 1.60 mm
- net PSU: track 81.8 -> 81.2 mm
Other:
- board text added: "CONTROELR V1.2"
- board text removed: "CONTROELR V1.1"
