File: HW/OCTO_CONTROLER_V1.2.sch (EAGLE design)
At the start: 44 parts, among them IC1 NTMD5838NL, IC2 NTMD5838NL, IC3 CXDM4060P, IC4 AOZ1284PI, J1 DC_POWER, Q1 DTC114EUA, Q2 CXDM4060P, Q3 DTC114EUA, X1 RASPI_BOARD_B+#_F

Commit message: BOM & V1.2 PCB UPDATE
Parts:
- added R14: 10kF, cona_lib:R_0603
- added ZD4, ZD5: RD36S, GRU-EURO6:ZENER_DIODERD47S
- added ZD6: RD16S, GRU-EURO6:ZENER_DIODERD47S
- R10: value 4.7k -> 47k
- R11: value 47k -> 2k
- R12: value 52.3kF -> 2.2k
- R13: value 10kF -> 52.3kF
- R9: value 10kF -> 10k
- ZD1: value SM6T39CAY -> SM6T33CAY
Connections:
- new net N$1: Q2.G, R11.1, R12.2, ZD6.A
- new net N$3: ZD4.A, ZD5.A
- net +5V: now also R13.2; no longer R12.2
- net GND: now also R10.2, R14.1; no longer R11.2, R13.1
- net N$12: now also R13.1, R14.2; no longer R12.1, R13.2
- net N$15: now also ZD5.C
- net N$28: now also R10.1; no longer R11.1
- net N$32: now also R12.1; no longer Q2.G, R10.1
- net VEE: now also R11.2, ZD4.C, ZD6.C; no longer R10.2
Other:
- note added: "2.54mm 12mm PIN HEADER SOCKET"
- note added: "DC7~30V Input range(DC 12V or DC24V)"
- note added: "OCTO PRINTER CONTROLER V1.2"
- note added: "RASPBERRY PI 3.5 " TFT LCD( 320*480) USED"
- note removed: "DC7~35V Input range(DC 12V or DC24V)"
- note removed: "OCTO PRINTER CONTROLER V1.1"
- moved on the sheet: D1, JP4, Q2, Q3, R10, R11, R12, R13
