File: HW/OCTO_CONTROLER_V1.3.brd (EAGLE design)
At the start: 65 x 56 mm, 64 parts, among them IC1 NTMD5838NL, IC2 NTMD5838NL, IC3 CXDM4060P, IC4 AOZ1284PI, IC5 NTMD5838NL, IC6 NTMD5838NL, J1 DC_POWER, Q1 DTC114EUA, Q2 CXDM4060P, Q3 DTC114EUA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

Commit message: V1.3 PCB PATHC
DHT-22 PULL-UP  10k->4.7K
Parts:
- R15: value 10k -> 4.7K
Changed lines of the file:
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@@
 <attribute name="VALUE" x="6.84" y="-6.311" size="0.7" layer="27" ratio="10"/>
 </element>
-<element name="R15" library="cona_lib" package="R0603" value="10k" x="2.5" y="-3.5" smashed="yes" rot="R90">
+<element name="R15" library="cona_lib" package="R0603" value="4.7K" x="2.5" y="-3.5" smashed="yes" rot="R90">
 <attribute name="NAME" x="1.699" y="-1.541" size="0.7" layer="25" rot="R180"/>
 <attribute name="VALUE" x="4.024" y="-5.024" size="0.7" layer="27" ratio="10" rot="R90"/>
